Commit message: Ready to collect data

File: blender_models/suzanne.urdf (robot description, URDF)
Before this commit: robot suzanne, 1 links, 0 joints
Links:
- removed link base_link
- added link suzanne, mass 1.0; collision mesh filename=suzanne_collision.obj scale=0.3770924 0.3770924 0.3770924; visual mesh filename=suzanne.obj scale=0.3770924 0.3770924 0.3770924
